Commit message: Updated URDF and launch file

File: src/robot_description/urdf/robot.urdf.xacro (robot description, xacro)
@@ -210,5 +210,5 @@
       <origin xyz="0 0 0" rpy="0 0 0"/>
       <geometry>
-        <box size="0.10 0.10 0.001"/>
+        <box size="0.25 0.25 0.001"/>
       </geometry>
       <material name="white"/>
@@ -217,5 +217,5 @@
       <origin xyz="0 0 0" rpy="0 0 0"/>
       <geometry>
-        <box size="0.10 0.10 0.001"/>
+        <box size="0.25 0.25 0.001"/>
       </geometry>
     </collision>
